Commit message: ros2 control 추가 및 모터 제어 추가

File: scara_description/urdf/scara_robot.urdf.xacro (robot description, xacro)
@@ -1,4 +1,21 @@
 <?xml version="1.0"?>
 <robot xmlns:xacro="[http://www.ros.org/wiki/xacro](http://www.ros.org/wiki/xacro)" name="scara_robot">
+    <xacro:arg name="use_sim" default="false"/>
+    <xacro:if value="$(arg use_sim)">
+        <ros2_control name="GazeboSystem" type="system">
+            <hardware>
+                <plugin>gazebo_ros2_control/GazeboSystem</plugin>
+            </hardware>
+            </ros2_control>
+    </xacro:if>
+    <xacro:unless value="$(arg use_sim)">
+        <ros2_control name="DynamixelSystem" type="system">
+            <hardware>
+                <plugin>ros_control_for_dynamixel/DynamixelSystemHardware</plugin>
+                <param name="usb_port">/dev/ttyUSB0</param>
+                <param name="baud_rate">57600</param>
+            </hardware>
+            </ros2_control>
+    </xacro:unless>
     <!-- 변수 및 재료 정의 -->
     <xacro:property name="link_1_length" value="0.2" />
@@ -11,7 +28,7 @@
     <link name="world" />
     <link name="base_link">
-        <visual><geometry><cylinder radius="0.05" length="0.1"/></geometry><material name="grey"/></visual>
-        <collision><geometry><cylinder radius="0.05" length="0.1"/></geometry></collision>
-        <inertial><mass value="1"/><inertia ixx="0.001" ixy="0" ixz="0" iyy="0.001" iyz="0" izz="0.001"/></inertial>
+        <visual><geometry><cylinder radius="0.05" length="0.1"/></geometry><material name="grey"/></visual><!--링크 비주얼-->
+        <collision><geometry><cylinder radius="0.05" length="0.1"/></geometry></collision><!--링크 충돌영역-->
+        <inertial><mass value="1"/><inertia ixx="0.001" ixy="0" ixz="0" iyy="0.001" iyz="0" izz="0.001"/></inertial><!--링크 물리적특성-->
     </link>
     <joint name="world_to_base" type="fixed"><parent link="world"/><child link="base_link"/><origin xyz="0 0 0.05" rpy="0 0 0"/></joint>
@@ -22,9 +39,9 @@
         <inertial><mass value="0.2"/><origin xyz="${link_1_length/2} 0 0" rpy="0 0 0"/><inertia ixx="0.000054" ixy="0.0" ixz="0.0" iyy="0.000694" iyz="0.0" izz="0.000694"/></inertial>
     </link>
-    <joint name="joint_1" type="revolute">
+    <joint name="joint_1" type="continuous">
         <parent link="base_link" /><child link="link_1" />
         <origin xyz="0 0 ${0.1/2}" rpy="0 0 0"/>
         <axis xyz="0 0 1"/>
-        <limit lower="-2.9" upper="2.9" effort="10" velocity="10"/>
+        <limit effort="1.5" velocity="6.38791"/>
     </joint>
     <transmission name="trans_1"><type>transmission_interface/SimpleTransmission</type><joint name="joint_1"><hardwareInterface>position</hardwareInterface></joint><actuator name="motor_1"><hardwareInterface>position</hardwareInterface></actuator></transmission>
@@ -35,9 +52,9 @@
         <inertial><mass value="0.2"/><origin xyz="${link_2_length/2} 0 0" rpy="0 0 0"/><inertia ixx="0.000054" ixy="0.0" ixz="0.0" iyy="0.000694" iyz="0.0" izz="0.000694"/></inertial>
     </link>
-    <joint name="joint_2" type="revolute">
-        <parent link="link_1" /><child link="link_2" />
-        <origin xyz="${link_1_length} 0 0"/>
+    <joint name="joint_2" type="continuous">
+        <parent link="base_link" /><child link="link_1" />
+        <origin xyz="0 0 ${0.1/2}" rpy="0 0 0"/>
         <axis xyz="0 0 1"/>
-        <limit lower="-2.9" upper="2.9" effort="10" velocity="10"/>
+        <limit effort="1.5" velocity="6.38791"/>
     </joint>
     <transmission name="trans_2"><type>transmission_interface/SimpleTransmission</type><joint name="joint_2"><hardwareInterface>position</hardwareInterface></joint><actuator name="motor_2"><hardwareInterface>position</hardwareInterface></actuator></transmission>
@@ -45,6 +62,8 @@
     <ros2_control name="GazeboSystem" type="system">
         <hardware><plugin>gazebo_ros2_control/GazeboSystem</plugin></hardware>
-        <joint name="joint_1"><command_interface name="position"><param name="min">-2.9</param><param name="max">2.9</param></command_interface><state_interface name="position"/><state_interface name="velocity"/></joint>
-        <joint name="joint_2"><command_interface name="position"><param name="min">-2.9</param><param name="max">2.9</param></command_interface><state_interface name="position"/><state_interface name="velocity"/></joint>
+        <joint name="joint_1"><command_interface name="velocity">
+        </command_interface><state_interface name="position"/><state_interface name="velocity"/></joint>
+        <joint name="joint_2"><command_interface name="velocity">
+        </command_interface><state_interface name="position"/><state_interface name="velocity"/></joint>
     </ros2_control>
     <gazebo>

Commit message: gazebo.launch 에러 수정 1차

File: scara_description/urdf/scara_robot.urdf.xacro (robot description, xacro)
@@ -39,9 +39,9 @@
         <inertial><mass value="0.2"/><origin xyz="${link_1_length/2} 0 0" rpy="0 0 0"/><inertia ixx="0.000054" ixy="0.0" ixz="0.0" iyy="0.000694" iyz="0.0" izz="0.000694"/></inertial>
     </link>
-    <joint name="joint_1" type="continuous">
+    <joint name="joint_1" type="revolute">
         <parent link="base_link" /><child link="link_1" />
         <origin xyz="0 0 ${0.1/2}" rpy="0 0 0"/>
         <axis xyz="0 0 1"/>
-        <limit effort="1.5" velocity="6.38791"/>
+        <limit lower="-3.14159" upper="3.14159" effort="1.5" velocity="6.38791"/>
     </joint>
     <transmission name="trans_1"><type>transmission_interface/SimpleTransmission</type><joint name="joint_1"><hardwareInterface>position</hardwareInterface></joint><actuator name="motor_1"><hardwareInterface>position</hardwareInterface></actuator></transmission>
@@ -52,18 +52,32 @@
         <inertial><mass value="0.2"/><origin xyz="${link_2_length/2} 0 0" rpy="0 0 0"/><inertia ixx="0.000054" ixy="0.0" ixz="0.0" iyy="0.000694" iyz="0.0" izz="0.000694"/></inertial>
     </link>
-    <joint name="joint_2" type="continuous">
-        <parent link="base_link" /><child link="link_1" />
-        <origin xyz="0 0 ${0.1/2}" rpy="0 0 0"/>
+    <joint name="joint_2" type="revolute">
+        <parent link="link_1" /><child link="link_2" />
+        <origin xyz="${link_1_length} 0 0" rpy="0 0 0"/>
         <axis xyz="0 0 1"/>
-        <limit effort="1.5" velocity="6.38791"/>
+        <limit lower="-3.14159" upper="3.14159" effort="1.5" velocity="6.38791"/>
     </joint>
     <transmission name="trans_2"><type>transmission_interface/SimpleTransmission</type><joint name="joint_2"><hardwareInterface>position</hardwareInterface></joint><actuator name="motor_2"><hardwareInterface>position</hardwareInterface></actuator></transmission>
     <!-- ROS2 CONTROL & GAZEBO PLUGIN -->
     <ros2_control name="GazeboSystem" type="system">
-        <hardware><plugin>gazebo_ros2_control/GazeboSystem</plugin></hardware>
-        <joint name="joint_1"><command_interface name="velocity">
-        </command_interface><state_interface name="position"/><state_interface name="velocity"/></joint>
-        <joint name="joint_2"><command_interface name="velocity">
-        </command_interface><state_interface name="position"/><state_interface name="velocity"/></joint>
+        <hardware>
+            <plugin>gazebo_ros2_control/GazeboSystem</plugin>
+        </hardware>
+        <joint name="joint_1">
+            <command_interface name="position">
+                <param name="min">-3.14159</param>
+                <param name="max">3.14159</param>
+            </command_interface>
+            <state_interface name="position"/>
+            <state_interface name="velocity"/>
+        </joint>
+        <joint name="joint_2">
+            <command_interface name="position"/>
+                <param name="min">-3.14159</param>
+                <param name="max">3.14159</param>
+            </command_interface>
+            <state_interface name="position"/>
+            <state_interface name="velocity"/>
+        </joint>
     </ros2_control>
     <gazebo>

Commit message: dynamixel packages add

File: scara_description/urdf/scara_robot.urdf.xacro (robot description, xacro)
@@ -2,4 +2,5 @@
 <robot xmlns:xacro="[http://www.ros.org/wiki/xacro](http://www.ros.org/wiki/xacro)" name="scara_robot">
     <xacro:arg name="use_sim" default="false"/>
+    <!--가상 gazebo ros2 control 설정-->
     <xacro:if value="$(arg use_sim)">
         <ros2_control name="GazeboSystem" type="system">
@@ -7,14 +8,51 @@
                 <plugin>gazebo_ros2_control/GazeboSystem</plugin>
             </hardware>
-            </ros2_control>
+            <joint name="joint_1">
+                <command_interface name="position">
+                    <param name="min">-3.14159</param>
+                    <param name="max">3.14159</param>
+                </command_interface>
+                <state_interface name="position"/>
+                <state_interface name="velocity"/>
+            </joint>
+            <joint name="joint_2">
+                <command_interface name="position">
+                    <param name="min">-3.14159</param>
+                    <param name="max">3.14159</param>
+                </command_interface>
+                <state_interface name="position"/>
+                <state_interface name="velocity"/>
+            </joint>
+        </ros2_control>
+        <gazebo>
+            <plugin name="gazebo_ros2_control" filename="libgazebo_ros2_control.so">
+                <parameters>$(find scara_description)/config/scara_controllers.yaml</parameters>
+            </plugin>
+        </gazebo>
+            <gazebo reference="link_1">
+                <disable_collisions link1="base_link" link2="link_1" />
+            </gazebo>
+        <gazebo reference="link_2">
+            <disable_collisions link1="link_1" link2="link_2" />
+        </gazebo>
     </xacro:if>
+    <!--실제 로봇 roe2 control 설정-->
     <xacro:unless value="$(arg use_sim)">
         <ros2_control name="DynamixelSystem" type="system">
             <hardware>
-                <plugin>ros_control_for_dynamixel/DynamixelSystemHardware</plugin>
-                <param name="usb_port">/dev/ttyUSB0</param>
-                <param name="baud_rate">57600</param>
+                <plugin>dynamixel_hardware_interface/DynamixelHardware</plugin>
+                <param name="dynamixel_info">$(find scara_description)/config/dynamixel_info.yaml</param>
             </hardware>
-            </ros2_control>
+            <joint name="joint_1">
+                <command_interface name="position"/>
+                <state_interface name="position"/>
+                <state_interface name="velocity"/>
+            </joint>
+            <joint name="joint_2">
+                <command_interface name="position"/>
+                <state_interface name="position"/>
+                <state_interface name="velocity"/>
+            </joint>
+        </ros2_control>
     </xacro:unless>
     <!-- 변수 및 재료 정의 -->
@@ -45,5 +83,4 @@
         <limit lower="-3.14159" upper="3.14159" effort="1.5" velocity="6.38791"/>
     </joint>
-    <transmission name="trans_1"><type>transmission_interface/SimpleTransmission</type><joint name="joint_1"><hardwareInterface>position</hardwareInterface></joint><actuator name="motor_1"><hardwareInterface>position</hardwareInterface></actuator></transmission>
     <!-- 링크 2 -->
     <link name="link_2">
@@ -58,37 +95,4 @@
         <limit lower="-3.14159" upper="3.14159" effort="1.5" velocity="6.38791"/>
     </joint>
-    <transmission name="trans_2"><type>transmission_interface/SimpleTransmission</type><joint name="joint_2"><hardwareInterface>position</hardwareInterface></joint><actuator name="motor_2"><hardwareInterface>position</hardwareInterface></actuator></transmission>
     <!-- ROS2 CONTROL & GAZEBO PLUGIN -->
-    <ros2_control name="GazeboSystem" type="system">
-        <hardware>
-            <plugin>gazebo_ros2_control/GazeboSystem</plugin>
-        </hardware>
-        <joint name="joint_1">
-            <command_interface name="position">
-                <param name="min">-3.14159</param>
-                <param name="max">3.14159</param>
-            </command_interface>
-            <state_interface name="position"/>
-            <state_interface name="velocity"/>
-        </joint>
-        <joint name="joint_2">
-            <command_interface name="position"/>
-                <param name="min">-3.14159</param>
-                <param name="max">3.14159</param>
-            </command_interface>
-            <state_interface name="position"/>
-            <state_interface name="velocity"/>
-        </joint>
-    </ros2_control>
-    <gazebo>
-        <plugin name="gazebo_ros2_control" filename="libgazebo_ros2_control.so">
-            <parameters>$(find scara_description)/config/scara_controllers.yaml</parameters>
-        </plugin>
-    </gazebo>
-    <gazebo reference="link_1">
-        <disable_collisions link1="base_link" link2="link_1" />
-    </gazebo>
-    <gazebo reference="link_2">
-        <disable_collisions link1="link_1" link2="link_2" />
-    </gazebo>
 </robot>

Commit message: git push 에러 수정

File: scara_description/urdf/scara_robot.urdf.xacro (robot description, xacro)
@@ -1,4 +1,4 @@
 <?xml version="1.0"?>
-<robot xmlns:xacro="[http://www.ros.org/wiki/xacro](http://www.ros.org/wiki/xacro)" name="scara_robot">
+<robot xmlns:xacro="http://www.ros.org/wiki/xacro" name="scara_robot">
     <xacro:arg name="use_sim" default="false"/>
     <!--가상 gazebo ros2 control 설정-->
@@ -38,8 +38,8 @@
     </xacro:if>
     <!--실제 로봇 roe2 control 설정-->
-    <xacro:unless value="$(arg use_sim)">
+    <!--<xacro:unless value="$(arg use_sim)">
         <ros2_control name="DynamixelSystem" type="system">
             <hardware>
-                <plugin>dynamixel_hardware_interface/DynamixelHardware</plugin>
+                <plugin>dynamixel_workbench/DynamixelWorkbench</plugin>
                 <param name="dynamixel_info">$(find scara_description)/config/dynamixel_info.yaml</param>
             </hardware>
@@ -54,4 +54,71 @@
                 <state_interface name="velocity"/>
             </joint>
+        </ros2_control>
+    </xacro:unless>-->
+    <xacro:unless value="$(arg use_sim)">
+        <ros2_control name="DynamixelSystem" type="system">
+            <hardware>
+                <plugin>dynamixel_hardware_interface/DynamixelHardware</plugin>
+                <param name="port_name">/dev/ttyUSB0</param>
+                <param name="baud_rate">57600</param>
+                <param name="error_timeout_ms">500</param>
+                <param name="number_of_joints">2</param>
+                <param name="number_of_transmissions">2</param>
+                <param name="dynamixel_model_folder">/param/dxl_model</param>
+                <param name="disable_torque_at_init">true</param>
+                <param name="transmission_to_joint_matrix">1,0,0,1</param>
+                <param name="joint_to_transmission_matrix">1,0,0,1</param>
+                <param name="dynamixel_state_pub_msg_name">dynamixel_hardware_interface/dxl_state</param>
+                <param name="get_dynamixel_data_srv_name">dynamixel_hardware_interface/get_dxl_data</param>
+                <param name="set_dynamixel_data_srv_name">dynamixel_hardware_interface/set_dxl_data</param>
+                <param name="reboot_dxl_srv_name">dynamixel_hardware_interface/reboot_dxl</param>
+                <param name="set_dxl_torque_srv_name">dynamixel_hardware_interface/set_dxl_torque</param>
+                </hardware>
+            <joint name="joint_1">
+                <command_interface name="position"/>
+                <state_interface name="position"/>
+                <state_interface name="velocity"/>
+            </joint>
+            <joint name="joint_2">
+                <command_interface name="position"/>
+                <state_interface name="position"/>
+                <state_interface name="velocity"/>
+            </joint>
+            <gpio name="joint_1_motor">
+                <param name="type">dxl</param>
+                <param name="ID">1</param>
+                <command_interface name="Goal Position"/>
+                <state_interface name="Present Position"/>
+                <state_interface name="Present Velocity"/>
+                <param name="Position P Gain">800</param>
+                <param name="Position I Gain">100</param>
+                <param name="Position D Gain">100</param>
+                <param name="Profile Velocity">200</param>
+                <param name="Profile Acceleration">50</param>
+                <param name="Drive Mode">1</param>
+            </gpio>
+            <gpio name="joint_2_motor">
+                <param name="type">dxl</param>
+                <param name="ID">2</param>
+                <command_interface name="Goal Position"/>
+                <state_interface name="Present Position"/>
+                <state_interface name="Present Velocity"/>
+                <param name="Position P Gain">800</param>
+                <param name="Position I Gain">100</param>
+                <param name="Position D Gain">100</param>
+                <param name="Profile Velocity">200</param>
+                <param name="Profile Acceleration">50</param>
+                <param name="Drive Mode">1</param>
+            </gpio>
+            <transmission name="tran1">
+                <plugin>transmission_interface/SimpleTransmissionLoader</plugin>
+                <joint name="joint_1" role="joint"/>
+                <actuator name="joint_1_motor" role="actuator"/>
+            </transmission>
+            <transmission name="tran2">
+                <plugin>transmission_interface/SimpleTransmissionLoader</plugin>
+                <joint name="joint_2" role="joint"/>
+                <actuator name="joint_2_motor" role="actuator"/>
+            </transmission>
         </ros2_control>
     </xacro:unless>
